File: main-board/main-board.kicad_pcb (KiCad board)
At the start: 2 copper layers, 180 x 111 mm, 53 parts, among them J1 INPUT, J2 NC1, J3 OUTPUT, J4 Conn_01x03_Pin, J5 COM, J6 Conn_01x03_Pin, SW1 SW_SPST, U1 ADA4898-2, U2 ADA4898-2, U3 AD633ANZ

Commit message: test gerber files and add JLC serial number to the main board
Other:
- board text added: "JLCJLCJLCJLC"
- board text added: "Serial Number:"
Changed lines of the file:
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@@
       (usegerberattributes true)
       (usegerberadvancedattributes true)
-      (creategerberjobfile true)
+      (creategerberjobfile false)
       (dashed_line_dash_ratio 12.000000)
       (dashed_line_gap_ratio 3.000000)
@@
       (outputformat 1)
       (mirror false)
-      (drillshape 1)
+      (drillshape 0)
       (scaleselection 1)
       (outputdirectory "")
@@
   (gr_arc (start 60 52) (mid 62.636039 45.636039) (end 69 43)
     (stroke (width 0.1) (type default)) (layer "Edge.Cuts"))
+  (gr_text "Serial Number:" (at 219.6 151.6) (layer "B.SilkS")
+    (effects (font (size 1 1) (thickness 0.2) bold) (justify left bottom mirror))
+  )
+  (gr_text "JLCJLCJLCJLC" (at 207.6 151.6) (layer "B.SilkS")
+    (effects (font (size 1 1) (thickness 0.2) bold) (justify left bottom mirror))
+  )
   (gr_text "Original Design from: 5-th Experimental Physics Olympiad (2017)\nAdapted by: Carlos Veras (@CarlosCraveiro - 2024)\nGitHub: https://github.com/CarlosCraveiro/einstein-boltzmann\n" (at 220 142.8) (layer "B.SilkS")
     (effects (font (size 2 2) (thickness 0.3) bold) (justify left bottom mirror))
