File: main-board/main-board.kicad_sch (KiCad schematic)
At the start: 52 parts, among them J4 Conn_01x03_Pin, J5 COM, J6 Conn_01x03_Pin, SW1 SW_SPST, U1 ADA4898-2, U2 ADA4898-2, U3 AD633ANZ

Commit message: Saves progress
Parts:
- added SW2, SW3: SW_Push_SPDT, symbol Switch:SW_Push_SPDT
- INPUT1, J5, NC1, OUTPUT1: footprint Connector_PinHeader_2.54mm:PinHeader_1x01_P2.54mm_Vertical -> footprints:Banana_Jack_1Pin
Changed lines of the file:
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@@
     (effects (font (size 2.5 2.5) bold) (justify left bottom))
   )
-  (text "M5" (at 232.41 138.43 0)
+  (text "M5" (at 224.79 153.67 0)
     (effects (font (size 1.27 1.27)) (justify left bottom))
   )
@@
     )
   )
+  (symbol (lib_id "Switch:SW_Push_SPDT") (at 188.595 139.7 0) (unit 1)
+    (in_bom yes) (on_board yes) (dnp no) (fields_autoplaced)
+    (property "Reference" "SW3" (at 188.595 130.81 0)
+      (effects (font (size 1.27 1.27)))
+    )
+    (property "Value" "SW_Push_SPDT" (at 188.595 133.35 0)
+      (effects (font (size 1.27 1.27)))
+    )
+    (property "Footprint" "" (at 188.595 139.7 0)
+      (effects (font (size 1.27 1.27)) hide)
+    )
+    (property "Datasheet" "~" (at 188.595 139.7 0)
+      (effects (font (size 1.27 1.27)) hide)
+    )
+    (pin "1")
+    (pin "2")
+    (pin "3")
+    (instances
+      (project "main-board"
+        (path "/99206265-9bbc-437e-9194-cd0123f9f5d5"
+          (reference "SW3") (unit 1)
+        )
+      )
+    )
+  )
   (symbol (lib_id "Device:C") (at 109.22 58.42 90) (unit 1)
     (in_bom yes) (on_board yes) (dnp no) (fields_autoplaced)
@@
         (path "/99206265-9bbc-437e-9194-cd0123f9f5d5"
           (reference "C1") (unit 1)
+        )
+      )
+    )
+  )
+  (symbol (lib_id "Switch:SW_Push_SPDT") (at 187.325 120.65 0) (unit 1)
+    (in_bom yes) (on_board yes) (dnp no) (fields_autoplaced)
+    (property "Reference" "SW2" (at 187.325 111.76 0)
+      (effects (font (size 1.27 1.27)))
+    )
+    (property "Value" "SW_Push_SPDT" (at 187.325 114.3 0)
+      (effects (font (size 1.27 1.27)))
+    )
+    (property "Footprint" "" (at 187.325 120.65 0)
+      (effects (font (size 1.27 1.27)) hide)
+    )
+    (property "Datasheet" "~" (at 187.325 120.65 0)
+      (effects (font (size 1.27 1.27)) hide)
+    )
+    (pin "1")
+    (pin "2")
+    (pin "3")
+    (instances
+      (project "main-board"
+        (path "/99206265-9bbc-437e-9194-cd0123f9f5d5"
+          (reference "SW2") (unit 1)
         )
       )
@@
       (effects (font (size 1.27 1.27)) (justify left))
     )
-    (property "Footprint" "Connector_PinHeader_2.54mm:PinHeader_1x01_P2.54mm_Vertical" (at 205.105 62.865 0)
+    (property "Footprint" "footprints:Banana_Jack_1Pin" (at 205.105 62.865 0)
       (effects (font (size 1.27 1.27)) hide)
     )
@@
       (effects (font (size 1.27 1.27)) (justify right))
     )
-    (property "Footprint" "Connector_PinHeader_2.54mm:PinHeader_1x01_P2.54mm_Vertical" (at 236.855 62.865 0)
+    (property "Footprint" "footprints:Banana_Jack_1Pin" (at 236.855 62.865 0)
       (effects (font (size 1.27 1.27)) hide)
     )
@@
       (effects (font (size 1.27 1.27)))
     )
-    (property "Footprint" "Connector_PinHeader_2.54mm:PinHeader_1x01_P2.54mm_Vertical" (at 71.755 140.335 0)
+    (property "Footprint" "footprints:Banana_Jack_1Pin" (at 71.755 140.335 0)
       (effects (font (size 1.27 1.27)) hide)
     )
@@
       (effects (font (size 1.27 1.27)))
     )
-    (property "Footprint" "Connector_PinHeader_2.54mm:PinHeader_1x01_P2.54mm_Vertical" (at 271.78 80.645 0)
-      (effects (font (size 1.27 1.27)) hide)
-    )
+    (property "Footprint" "footprints:Banana_Jack_1Pin" (at 271.78 80.645 0)
+      (effects (font (size 1.27 1.27)) hide)
+    )
